Commit message: tetra_description 수정

File: tetra_description/urdf/base.urdf.xacro (robot description, xacro)
@@ -2,108 +2,68 @@
 <robot name="tetra" xmlns:xacro="http://ros.org/wiki/xacro">
   <!-- Define a number of dimensions using properties -->
-  <xacro:property name="base_length" value="0.473" />
-  <xacro:property name="base_radius" value="0.2365" />
-  <xacro:property name="wheel_length" value="0.047" />
-  <xacro:property name="wheel_radius" value="0.085" />
+  <xacro:property name="base_length" value="0.492" />
+  <xacro:property name="base_radius" value="0.460" />
   <xacro:property name="wheel_offset_x" value="0.0" />
-  <xacro:property name="wheel_offset_y" value="0.1975" /> <!--0.220-->
-  <xacro:property name="wheel_offset_z" value="-0.100" />
-  <xacro:property name="PI" value="3.1415926" />
-  <xacro:macro name="cylinder_inertia" params="m r h">
-        <inertia ixx="${m*(3*r*r+h*h)/12}" ixy="0" ixz="0" iyy="${m*(3*r*r+h*h)/12}" iyz="0" izz="${m*r*r/2}" />
-  </xacro:macro>
+  <xacro:property name="wheel_offset_y" value="0.1975" />
+  <xacro:property name="wheel_offset_z" value="0" />
   <!-- define a wheel -->
   <joint name="base_l_wheel_joint" type="fixed">
     <axis xyz="0 1 0" />
-    <origin xyz="${wheel_offset_x} ${wheel_offset_y} 0" rpy="0 0 0" />
-    <parent link="base_link"/>
-    <child link="base_l_wheel_link"/>
-   </joint>
-    <link name="base_l_wheel_link">
-    </link>
- <joint name="base_r_wheel_joint" type="fixed">
+    <origin xyz="${wheel_offset_x} ${wheel_offset_y} ${wheel_offset_z}" rpy="0 0 0" />
+    <parent link="base_link" />
+    <child link="base_l_wheel_link" />
+  </joint>
+  <link name="base_l_wheel_link" />
+  <joint name="base_r_wheel_joint" type="fixed">
     <axis xyz="0 1 0" />
-    <origin xyz="${wheel_offset_x} ${-1.0*wheel_offset_y} 0" rpy="0 0 0" />
-    <parent link="base_link"/>
-    <child link="base_r_wheel_link"/>
-   </joint>
-    <link name="base_r_wheel_link">
-    </link>
+    <origin xyz="${wheel_offset_x} ${-wheel_offset_y} ${wheel_offset_z}" rpy="0 0 0" />
+    <parent link="base_link" />
+    <child link="base_r_wheel_link" />
+  </joint>
+  <link name="base_r_wheel_link" />
   <!-- The base xacro macro -->
-   <link name="base_link">
+  <link name="base_link">
     <visual>
-    <origin xyz=" 0 0 0 " rpy="0 0 0" />
+      <origin xyz=" 0 0 0 " rpy="0 0 0" />
       <geometry>
-        <mesh
-          filename="package://tetra_description/meshes/tetra_dsv_sm.stl" scale="0.001 0.001 0.001" />
+        <mesh filename="package://tetra_description/meshes/tetra_dsv_edu.stl" scale="0.001 0.001 0.001" />
       </geometry>
-      <material name="black"/>
+      <material name="black" />
     </visual>
-      <collision>
-            <origin xyz="0 0 0" rpy="0 0 0"/>
-            <geometry>
-                <cylinder length="${base_length}" radius="${base_radius}"/>
-            </geometry>
-      </collision>
-    </link>
+    <collision>
+      <origin xyz="0 0 0" rpy="0 0 0" />
+      <geometry>
+        <mesh filename="package://tetra_description/meshes/tetra_dsv_edu.stl" scale="0.001 0.001 0.001" />
+      </geometry>
+    </collision>
+  </link>
   <link name="base_footprint">
-      <visual>
-        <origin xyz="-0.104 0 0" rpy="0 0 0" />
-        <geometry>
-	  <box size="0.492 0.460 0.001" />
-        </geometry>
-        <material name="transparentgreen" />
-      </visual>
+    <visual>
+      <origin xyz="-0.104 0 0" rpy="0 0 0" />
+      <geometry>
+	      <box size="${base_length} ${base_radius} 0.001" />
+      </geometry>
+      <material name="transparentgreen" />
+    </visual>
   </link>
-  <joint name="base_joint" type="fixed"> <!--fixed-->
-    <origin xyz="0 0 ${-wheel_offset_z}" rpy="0 0 0" />
-    <parent link="base_footprint"/>
+  <joint name="base_joint" type="fixed">
+    <origin xyz="0 0 0.1" rpy="0 0 0" />
+    <parent link="base_footprint" />
     <child link="base_link" />
   </joint>
   <!-- Rear Caster-->
-  <xacro:macro name="rear_caster_wheel" params="prefix dir">
-        <link name="${prefix}_rear_caster_rotate">
-            <collision>
-                <origin xyz="0 0 0" rpy="0 0 0"/>
-                <geometry>
-                    <mesh filename="package://tetra_description/meshes/caster_yoke.stl" scale="0.001 0.001 0.001" />
-                </geometry>
-            </collision>
-            <inertial>
-                <mass value="0.1"/>
-                <origin xyz="0 0 0" rpy="0 0 0"/>
-                <xacro:cylinder_inertia m="0.1" r="0.03" h="0.03"/>
-            </inertial>
-        </link>
-        <joint name="${prefix}_rear_caster_rotate_joint" type="fixed">
-            <parent link="base_link"/>
-            <child link="${prefix}_rear_caster_rotate"/>
-            <origin xyz="-0.281 0 0.00303" rpy="0 0 0"/> <!-- -0.300 ${dir*-0.160} -0.0225 ... 230630 mwcha -->
-            <axis xyz="0 0 1"/>
-        </joint>
-        <link name="${prefix}_rear_caster_wheel">
-            <collision>
-                <origin xyz="0 0 0" rpy="0 0 0"/>
-                <geometry>
-                    <mesh filename="package://tetra_description/meshes/caster_wheel.stl" scale="0.001 0.001 0.001" />
-                </geometry>
-            </collision>
-            <inertial>
-                <mass value="0.1"/>
-                <origin xyz="0 0 0" rpy="${PI/2} 0 0"/>
-                <xacro:cylinder_inertia m="0.1" r="0.06" h="0.04"/>
-            </inertial>
-        </link>
-        <joint name="${prefix}_rear_caster_wheel_joint" type="fixed">
-            <parent link="${prefix}_rear_caster_rotate"/>
-            <child link="${prefix}_rear_caster_wheel"/>
-            <origin xyz="-0.022 0 -0.04632" rpy="0 0 0"/> <!-- -0.022 0 -0.047 ... 230630 mwcha -->
-            <axis xyz="0 1 0"/>
-        </joint>
-    </xacro:macro>
-  <xacro:rear_caster_wheel prefix="l" dir="1"/>
-<!--
-  <xacro:rear_caster_wheel prefix="r" dir="-1"/>
-230630 mwcha
--->
+  <joint name="rear_caster_rotate_joint" type="fixed">
+    <parent link="base_link" />
+    <child link="rear_caster_rotate" />
+    <origin xyz="-0.281 0 0.00303" rpy="0 0 0" />
+    <axis xyz="0 0 1" />
+  </joint>
+  <link name="rear_caster_rotate" />
+  <joint name="rear_caster_wheel_joint" type="fixed">
+    <parent link="rear_caster_rotate" />
+    <child link="rear_caster_wheel" />
+    <origin xyz="-0.022 0 -0.04632" rpy="0 0 0" />
+    <axis xyz="0 1 0" />
+  </joint>
+  <link name="rear_caster_wheel" />
 </robot>

File: tetra_description/urdf/tetra.xacro (robot description, xacro)
@@ -2,144 +2,27 @@
 <robot name="tetra" xmlns:xacro="http://ros.org/wiki/xacro">
   <!-- Define a number of dimensions using properties -->
-  <xacro:property name="base_length" value="0.473" />
-  <xacro:property name="base_radius" value="0.2365" />
-  <xacro:property name="wheel_length" value="0.047" />
-  <xacro:property name="wheel_radius" value="0.085" />
-  <xacro:property name="wheel_offset_x" value="0.0" />
-  <xacro:property name="wheel_offset_y" value="0.207" /> <!--0.220-->
-  <xacro:property name="wheel_offset_z" value="-0.100" />
   <xacro:property name="PI" value="3.1415926" />
-  <xacro:macro name="cylinder_inertia" params="m r h">
-        <inertia ixx="${m*(3*r*r+h*h)/12}" ixy="0" ixz="0" iyy="${m*(3*r*r+h*h)/12}" iyz="0" izz="${m*r*r/2}" />
-  </xacro:macro>
-   <!-- Include all component files -->
-   <xacro:include filename="$(find tetra_description)/urdf/materials.urdf.xacro" />
-   <xacro:include filename="$(find tetra_description)/urdf/base.urdf.xacro" />
-   <!-- Add the base and wheels -->
-   <base name="base" color="black"/>
-  <link name="laser">
-      <visual>
-        <origin xyz="0 0 0" rpy="0 0 0" />
-        <geometry>
-          <box size="0.01 0.01 0.01" />
-        </geometry>
-        <material name="grey" />
-      </visual>
-  </link>
-  <joint name="laser_flag" type="fixed">
-    <!--<origin xyz="0.060 0 0.210" rpy="0 0 -0.296706" />-->
-    <!--<origin xyz="0.060 0 0.210" rpy="0 0 -1.57079632679" />-->
-    <origin xyz="0.060 0 0.210" rpy="0 0 0" />
+  <!-- Include all component files -->
+  <xacro:include filename="$(find tetra_description)/urdf/materials.urdf.xacro" />
+  <xacro:include filename="$(find tetra_description)/urdf/base.urdf.xacro" />
+  <!-- Add the base and wheels -->
+  <base name="base" color="black"/>
+  <joint name="lidar" type="fixed">
+    <origin xyz="0.045 0 0.17" rpy="0 0 ${-PI/2}" />
+    <parent link="base_link" />
+    <child link="lidar_link" />
+  </joint>
+  <link name="lidar_link" />
+  <joint name="camera" type="fixed">
+    <origin xyz="0.109 0.03 0.125" rpy="0 0 0"/>
     <parent link="base_link"/>
-    <child link="laser" />
+    <child link="camera_link" />
   </joint>
-  <link name="laser_link2">
-      <visual>
-        <origin xyz="0 0 0" rpy="0 0 0" />
-        <geometry>
-          <box size="0.01 0.01 0.01" />
-        </geometry>
-        <material name="grey" />
-      </visual>
-  </link>
-  <joint name="base_link_to_laser_link2" type="fixed">
-    <origin xyz="-0.350 0.0 0.2436" rpy="0 0 ${PI}" />
+  <link name="camera_link" />
+  <joint name="front_bumper" type="fixed">
+    <origin xyz="0.142 0.0 -0.025" rpy="0 0 0" />
     <parent link="base_link"/>
-    <child link="laser_link2" />
+    <child link="front_bumper_link" />
   </joint>
-  <link name="imu_link">
-      <visual>
-        <origin xyz="0 0 0" rpy="0 0 0" />
-        <geometry>
-          <box size="0.01 0.01 0.01" />
-        </geometry>
-        <material name="grey" />
-      </visual>
-  </link>
-  <joint name="base_link_to_imu_link" type="fixed">
-    <origin xyz="-0.025 0 0.232" rpy="0 0 0" />
-    <parent link="base_link"/>
-    <child link="imu_link" />
-  </joint>
- <link name="camera">
-      <visual>
-        <origin xyz="0 0 0" rpy="0 0 0" />
-        <geometry>
-          <box size="0.01 0.01 0.01" />
-        </geometry>
-        <material name="grey" />
-      </visual>
-  </link>
-  <joint name="camera" type="fixed">
-    <origin xyz="0.11 0.0 0.181" rpy="1.5708 3.14159 1.5708"/>
-    <parent link="base_link"/>
-    <child link="camera" />
-  </joint>
- <link name="front_bumper">
-      <visual>
-        <origin xyz="0 0 0" rpy="0 0 0" />
-        <geometry>
-          <box size="0.01 0.30 0.01" />
-        </geometry>
-        <material name="transparentblack" />
-      </visual>
-  </link>
-  <joint name="front_bumper" type="fixed">
-    <origin xyz="0.12625 0.0 -0.05" rpy="0 0 0" />
-    <parent link="base_link"/>
-    <child link="front_bumper" />
-  </joint>
-  <link name="camera1_link">
-      <visual>
-        <origin xyz="0 0 0" rpy="0 0 0" />
-        <geometry>
-          <box size="0.01 0.01 0.01" />
-        </geometry>
-        <material name="grey" />
-      </visual>
-  </link>
-  <joint name="camera1_link" type="fixed">
-    <origin xyz="0.1097 0.015 0.1344" rpy="0 0 -0.0174" />
-    <parent link="base_link"/>
-    <child link="camera1_link" />
-  </joint>
-<!--
-   <link name="livox_frame">
-      <visual>
-        <origin xyz="0 0 0" rpy="0 0 0" />
-        <geometry>
-          <box size="0.01 0.01 0.01" />
-        </geometry>
-        <material name="grey" />
-      </visual>
-  </link>
-  <joint name="base_link_to_livox_frame" type="fixed">
-    <origin xyz="-0.0915 0.0 0.404" rpy="0 0 0"/>
-    <parent link="base_link"/>
-    <child link="livox_frame" />
-  </joint>
--->
-<!--
- <link name="base_upperlink">
-   <visual>
-    <origin xyz=" 0 0 0 " rpy="0 0 0" />
-      <geometry>
-        <mesh
-          filename="package://tetra_description/meshes/platform_body_u.stl" scale="0.001 0.001 0.001" />
-      </geometry>
-      <material name="transparentred"/>
-    </visual>
-      <collision>
-            <origin xyz="0 0 0" rpy="0 0 0"/>
-            <geometry>
-                <cylinder length="${base_length}" radius="${base_radius}"/>
-            </geometry>
-      </collision>
-  </link>
-  <joint name="base_upperlink" type="fixed">
-    <origin xyz="0.0 0.0 0.0" rpy="0 0 0" />
-    <parent link="base_link"/>
-    <child link="base_upperlink" />
-  </joint>
--->
+  <link name="front_bumper_link" />
 </robot>
