Commit message: 도킹 가운데로 들어가도록 수정

File: tetra_description/urdf/tetra.xacro (robot description, xacro)
@@ -15,5 +15,6 @@
   <link name="lidar_link" />
   <joint name="camera" type="fixed">
-    <origin xyz="0.109 0.03 0.125" rpy="0 0 0"/>
+    <!-- camera_link = D435 depth 원점. 컬러 센서(y=0.03)는 드라이버가 camera_link→camera_color_frame (y=+0.015)로 추가 -->
+    <origin xyz="0.109 0.015 0.125" rpy="0 0 0"/>
     <parent link="base_link"/>
     <child link="camera_link" />
